Commit message: measured real truck trailer

File: truck_trailer_sim/urdf/truck_trailer_prev.urdf (robot description, URDF)
Before this commit: robot truck_trailer, 9 links, 8 joints
Links:
- link trailer_link: geometry visual box size=0.555 0.35 0.08
- link truck_base: geometry visual box size=0.55 0.35 0.05
- link truck_cube: geometry visual box size=0.15 0.35 0.10
Joints:
- joint front_wheel_joint: origin xyz=0.4 0 0.04 rpy=0 0 0 -> xyz=0.3715 0 0.04 rpy=0 0 0
- joint hitch_joint: origin xyz=0.537 0 0 rpy=0 0 0 -> xyz=0.495 0 0 rpy=0 0 0
- joint rear_left_wheel_joint: origin xyz=-0.02 0.1275 0.04 rpy=0 0 0 -> xyz=-0.0495 0.135 0.04 rpy=0 0 0
- joint rear_right_wheel_joint: origin xyz=-0.02 -0.1275 0.04 rpy=0 0 0 -> xyz=-0.0495 -0.135 0.04 rpy=0 0 0
- joint trailer_left_wheel_joint: origin xyz=0 0.1225 0.04 rpy=0 0 0 -> xyz=0 0.135 0.04 rpy=0 0 0
- joint trailer_right_wheel_joint: origin xyz=0 -0.1225 0.04 rpy=0 0 0 -> xyz=0 -0.135 0.04 rpy=0 0 0
